File: hardware/kbxBinaryClock.v2.1/kbxBinaryClock-Display.v2.1.sch (KiCad schematic (older format))
At the start: 54 parts, among them Q10 Q_NPN_BCE, Q11 Q_NPN_BCE, Q6 Q_NPN_BCE, Q7 Q_NPN_BCE, Q8 Q_NPN_BCE, Q9 Q_NPN_BCE, U2 TLC5947, U3 TLC5947, U4 TLC5947

Commit message: Updated for KiCad v5, updated silks
Parts:
- C17, C18, C19: symbol C -> Device:C
- LED1, LED10, LED11, LED12, LED13, LED14, LED15, LED16, LED17, LED18, LED19, LED2, LED20, LED21, LED22, LED23, LED24, LED3, LED4, LED5, LED6, LED7, LED8, LED9: symbol LED_RGB_COMMON_ANODE -> win:LED_RGB_COMMON_ANODE
- Q10, Q11, Q6, Q7, Q8, Q9: symbol Q_NPN_BCE -> Device:Q_NPN_BCE
- R20, R21, R22, R23, R24, R25, R26, R27, R28, R29, R30, R31, R32, R33, R34, R35, R36, R37: symbol R -> Device:R
- U2, U3, U4: symbol TLC5947 -> win:TLC5947
