File: hardware/kbxBinaryClock.v2.1/kbxBinaryClock-MCU.v2.1.sch (KiCad schematic (older format))
At the start: 56 parts, among them P1 STM32_SWD_USART, Q1 2N7002, Q2 2N7002, Q3 2N7002, Q4 2N7002, Q5 Q_Photo_NPN, SW1 SW_Push, U1 STM32F072CBTx, Y1 32.768 KHz, Y2 8 MHz

Commit message: Modified PCBs to accommodate a 16mm buzzer element
Connections:
- net GND: now also RV1.3
Changed lines of the file:
@@
 Connection ~ 4350 1400
 Wire Wire Line
-	4600 1400 4350 1400
+	4200 1400 4600 1400
 Wire Wire Line
 	4350 1250 4350 1450
@@
 Wire Wire Line
 	9700 5100 9900 5100
+Wire Wire Line
+	4200 1100 4200 1400
 $EndSCHEMATC

Commit message: Added BoM, hw README, PCB tweaks
Parts:
- added D1: 1N4148, Diodes_SMD:D_SOD-123, symbol D
Connections:
- net +9V: now also D1.1 (K)
- net at BZ1.2 (+), Q1.3 (D): now also D1.2 (A)
Other:
- note added: "Install LED25 *OR* LED26\nDO NOT INSTALL BOTH"
Changed lines of the file:
@@
 Wire Wire Line
 	4200 1100 4200 1400
+$Comp
+L D D1
+U 1 1 5A896423
+P 1400 6150
+F 0 "D1" H 1400 6250 50  0000 C CNN
+F 1 "1N4148" H 1400 6050 50  0000 C CNN
+F 2 "Diodes_SMD:D_SOD-123" H 1400 6150 50  0001 C CNN
+F 3 "" H 1400 6150 50  0001 C CNN
+	1    1400 6150
+	0    1    1    0
+$EndComp
+Wire Wire Line
+	1400 6000 1400 5900
+Connection ~ 1400 5900
+Wire Wire Line
+	1400 6300 1400 6450
+Wire Wire Line
+	1400 6450 1250 6450
+Connection ~ 1250 6450
+Text Notes 2000 5800 0    60   ~ 0
+Install LED25 *OR* LED26\nDO NOT INSTALL BOTH
 $EndSCHEMATC

Commit message: Updated for KiCad v5, updated silks
Parts:
- BZ1: symbol Buzzer -> Device:Buzzer
- C1, C10, C11, C12, C13, C14, C15, C16, C2, C3, C4, C5, C6, C7, C8, C9: symbol C -> Device:C
- D1: symbol D -> Device:D
- LED25: symbol LED_RGB_COMMON_ANODE -> win:LED_RGB_COMMON_ANODE
- LED26: symbol LED_Dual_AACC -> Device:LED_Dual_AACC
- P1: symbol STM32_SWD_USART -> win:STM32_SWD_USART
- Q1, Q2, Q3, Q4: symbol 2N7002 -> kbxBinaryClock.v2.1-rescue:2N7002
- Q5: symbol Q_Photo_NPN -> Device:Q_Photo_NPN
- R1, R10, R11, R12, R13, R14, R15, R16, R17, R18, R19, R2, R3, R4, R5, R6, R7, R8, R9: symbol R -> Device:R
- RV1: symbol POT -> kbxBinaryClock.v2.1-rescue:POT
- SB1: symbol GS3 -> win:GS3
- SW1: symbol SW_Push -> kbxBinaryClock.v2.1-rescue:SW_Push
- TP1, TP2, TP3, TP4, TP5, TP6: symbol Conn_01x01 -> kbxBinaryClock.v2.1-rescue:Conn_01x01
- U1: symbol STM32F072CBTx -> kbxBinaryClock.v2.1-rescue:STM32F072CBTx
- Y1, Y2: symbol Crystal -> Device:Crystal
