File: hardware/kbxBinaryClock.v2.1/kbxBinaryClock-Peripherals.v2.1.sch (KiCad schematic (older format))
At the start: 14 parts, among them J2 Conn_01x06, J3 Conn_02x03_Odd_Even, U6 DS3231, U7 DS1621, U8 MAX485E

Commit message: Added BoM, hw README, PCB tweaks
Parts:
- removed R38: 10K, Resistors_SMD:R_0805, symbol R
- renumbered R39 to R38, R40 to R39, R41 to R40, R42 to R41
Changed lines of the file:
@@
 $EndComp
 $Comp
-L R R41
+L R R40
 U 1 1 5A0B2F28
 P 3150 1600
-F 0 "R41" V 3230 1600 50  0000 C CNN
+F 0 "R40" V 3230 1600 50  0000 C CNN
 F 1 "10K" V 3150 1600 50  0000 C CNN
 F 2 "Resistors_SMD:R_0805" V 3080 1600 50  0001 C CNN
@@
 $EndComp
 $Comp
-L R R38
-U 1 1 5A0B30BE
-P 2150 2700
-F 0 "R38" V 2230 2700 50  0000 C CNN
-F 1 "10K" V 2150 2700 50  0000 C CNN
-F 2 "Resistors_SMD:R_0805" V 2080 2700 50  0001 C CNN
-F 3 "" H 2150 2700 50  0001 C CNN
-	1    2150 2700
-	0    -1   -1   0
-$EndComp
-$Comp
-L +3.3V #PWR040
-U 1 1 5A0B3116
-P 1900 2700
-F 0 "#PWR040" H 1900 2550 50  0001 C CNN
-F 1 "+3.3V" H 1900 2840 50  0000 C CNN
-F 2 "" H 1900 2700 50  0001 C CNN
-F 3 "" H 1900 2700 50  0001 C CNN
-	1    1900 2700
-	1    0    0    -1
-$EndComp
-$Comp
-L R R40
+L R R39
 U 1 1 5A0B3562
 P 2400 1750
-F 0 "R40" V 2480 1750 50  0000 C CNN
+F 0 "R39" V 2480 1750 50  0000 C CNN
 F 1 "3K3" V 2400 1750 50  0000 C CNN
 F 2 "Resistors_SMD:R_0805" V 2330 1750 50  0001 C CNN
@@
 $EndComp
 $Comp
-L R R39
+L R R38
 U 1 1 5A0B35AA
 P 2200 1750
-F 0 "R39" V 2280 1750 50  0000 C CNN
+F 0 "R38" V 2280 1750 50  0000 C CNN
 F 1 "3K3" V 2200 1750 50  0000 C CNN
 F 2 "Resistors_SMD:R_0805" V 2130 1750 50  0001 C CNN
@@
 $EndComp
 $Comp
-L GND #PWR041
+L GND #PWR040
 U 1 1 5A0B3A49
 P 9000 3200
-F 0 "#PWR041" H 9000 2950 50  0001 C CNN
+F 0 "#PWR040" H 9000 2950 50  0001 C CNN
 F 1 "GND" H 9000 3050 50  0000 C CNN
 F 2 "" H 9000 3200 50  0001 C CNN
@@
 $EndComp
 $Comp
-L +3.3V #PWR042
+L +3.3V #PWR041
 U 1 1 5A0B3ACB
 P 9000 1700
-F 0 "#PWR042" H 9000 1550 50  0001 C CNN
+F 0 "#PWR041" H 9000 1550 50  0001 C CNN
 F 1 "+3.3V" H 9000 1840 50  0000 C CNN
 F 2 "" H 9000 1700 50  0001 C CNN
@@
 $EndComp
 $Comp
-L GND #PWR043
+L GND #PWR042
 U 1 1 5A0B3BC0
 P 9700 1900
-F 0 "#PWR043" H 9700 1650 50  0001 C CNN
+F 0 "#PWR042" H 9700 1650 50  0001 C CNN
 F 1 "GND" H 9700 1750 50  0000 C CNN
 F 2 "" H 9700 1900 50  0001 C CNN
@@
 $EndComp
 $Comp
-L GND #PWR044
+L GND #PWR043
 U 1 1 5A0B4904
 P 5850 2800
-F 0 "#PWR044" H 5850 2550 50  0001 C CNN
+F 0 "#PWR043" H 5850 2550 50  0001 C CNN
 F 1 "GND" H 5850 2650 50  0000 C CNN
 F 2 "" H 5850 2800 50  0001 C CNN
@@
 $EndComp
 $Comp
-L +3.3V #PWR045
+L +3.3V #PWR044
 U 1 1 5A0B49D6
 P 4900 1800
-F 0 "#PWR045" H 4900 1650 50  0001 C CNN
+F 0 "#PWR044" H 4900 1650 50  0001 C CNN
 F 1 "+3.3V" H 4900 1940 50  0000 C CNN
 F 2 "" H 4900 1800 50  0001 C CNN
@@
 Text HLabel 8400 2600 0    60   Input ~ 0
 USART2_TX
-Wire Wire Line
-	1150 2400 2400 2400
-Wire Wire Line
-	1150 2500 2400 2500
-Wire Wire Line
-	2900 1500 2900 2000
-Wire Wire Line
-	2100 1600 3000 1600
-Connection ~ 2900 1600
-Wire Wire Line
-	3800 2700 3800 1500
-Wire Wire Line
-	3400 2700 3800 2700
-Wire Wire Line
-	2900 3200 2900 3000
-Wire Wire Line
-	1700 1600 1800 1600
-Wire Wire Line
-	2300 2700 2400 2700
-Wire Wire Line
-	2400 2400 2400 1900
-Wire Wire Line
-	2200 1900 2200 2000
-Wire Wire Line
-	2200 2000 2300 2000
-Wire Wire Line
-	2300 2000 2300 2500
-Connection ~ 2300 2500
-Connection ~ 2400 1600
-Connection ~ 2200 1600
-Wire Wire Line
-	9400 2600 9800 2600
-Wire Wire Line
-	9400 2300 10400 2300
-Wire Wire Line
-	9600 2300 9600 2700
-Wire Wire Line
-	9600 2700 9800 2700
-Wire Wire Line
-	9000 3000 9000 3200
-Wire Wire Line
-	9800 2800 9600 2800
-Wire Wire Line
-	9600 2800 9600 3100
-Wire Wire Line
-	9000 3100 10300 3100
-Connection ~ 9000 3100
-Wire Wire Line
-	9000 1700 9000 1900
-Wire Wire Line
-	9300 1800 9000 1800
-Connection ~ 9000 1800
-Wire Wire Line
-	9600 1800 9700 1800
-Wire Wire Line
-	9700 1800 9700 1900
-Wire Wire Line
-	8600 2400 8600 2500
-Wire Wire Line
-	5850 2800 5850 2700
-Wire Wire Line
-	5850 2700 5950 2700
-Wire Wire Line
-	1900 2700 2000 2700
-Wire Wire Line
-	8400 2300 8600 2300
-Wire Wire Line
-	8600 2400 8400 2400
-Wire Wire Line
-	8400 2600 8600 2600
 $Comp
 L Conn_02x03_Odd_Even J3
@@
 	1    0    0    1
 $EndComp
-Wire Wire Line
-	10300 3100 10300 2800
-Connection ~ 9600 3100
-Wire Wire Line
-	10300 2600 10300 2450
-Wire Wire Line
-	10300 2450 9800 2450
-Wire Wire Line
-	9800 2450 9800 2600
-Wire Wire Line
-	10300 2700 10400 2700
-Wire Wire Line
-	10400 2700 10400 2300
-Connection ~ 9600 2300
 $Comp
 L C C25
@@
 	-1   0    0    1
 $EndComp
-Wire Wire Line
-	5400 1900 5800 1900
-Wire Wire Line
-	5800 2200 5950 2200
-Wire Wire Line
-	5600 2300 5950 2300
-Wire Wire Line
-	5950 2400 5600 2400
-Wire Wire Line
-	4900 1800 4900 2500
-Wire Wire Line
-	4900 2500 5950 2500
 $Comp
 L DS1621 U7
@@
 	1    0    0    -1
 $EndComp
-Wire Wire Line
-	2050 5100 1400 5100
-Wire Wire Line
-	1400 5100 1400 2400
-Connection ~ 1400 2400
-Wire Wire Line
-	2050 4900 1600 4900
-Wire Wire Line
-	1600 4900 1600 2500
-Connection ~ 1600 2500
-$Comp
-L +3.3V #PWR046
+$Comp
+L +3.3V #PWR045
 U 1 1 5A6AC87F
 P 2900 4250
-F 0 "#PWR046" H 2900 4100 50  0001 C CNN
+F 0 "#PWR045" H 2900 4100 50  0001 C CNN
 F 1 "+3.3V" H 2900 4390 50  0000 C CNN
 F 2 "" H 2900 4250 50  0001 C CNN
@@
 	1    0    0    -1
 $EndComp
-Wire Wire Line
-	2900 4600 2900 4250
 $Comp
 L C C24
@@
 $EndComp
 $Comp
-L GND #PWR047
+L GND #PWR046
 U 1 1 5A6ACBF8
 P 3850 4800
-F 0 "#PWR047" H 3850 4550 50  0001 C CNN
+F 0 "#PWR046" H 3850 4550 50  0001 C CNN
 F 1 "GND" H 3850 4650 50  0000 C CNN
 F 2 "" H 3850 4800 50  0001 C CNN
@@
 	1    0    0    -1
 $EndComp
-Wire Wire Line
-	2900 4400 3850 4400
-Wire Wire Line
-	3850 4400 3850 4450
-Connection ~ 2900 4400
-Wire Wire Line
-	3850 4750 3850 4800
-$Comp
-L GND #PWR048
+$Comp
+L GND #PWR047
 U 1 1 5A6ACE92
 P 2900 5900
-F 0 "#PWR048" H 2900 5650 50  0001 C CNN
+F 0 "#PWR047" H 2900 5650 50  0001 C CNN
 F 1 "GND" H 2900 5750 50  0000 C CNN
 F 2 "" H 2900 5900 50  0001 C CNN
@@
 	1    0    0    -1
 $EndComp
-Wire Wire Line
-	2900 5900 2900 5800
-Wire Wire Line
-	2050 5400 2050 5850
-Wire Wire Line
-	2050 5850 2900 5850
-Connection ~ 2900 5850
-Connection ~ 2050 5600
-Connection ~ 2050 5500
-Wire Wire Line
-	3400 2500 3600 2500
-Wire Wire Line
-	3600 2500 3600 1500
-Wire Wire Line
-	3300 1600 3600 1600
-Connection ~ 3600 1600
-$Comp
-L R R42
+$Comp
+L R R41
 U 1 1 5A800EAE
 P 3150 1800
-F 0 "R42" V 3230 1800 50  0000 C CNN
+F 0 "R41" V 3230 1800 50  0000 C CNN
 F 1 "10K" V 3150 1800 50  0000 C CNN
 F 2 "Resistors_SMD:R_0805" V 3080 1800 50  0001 C CNN
@@
 	0    -1   -1   0
 $EndComp
+Text HLabel 1150 2700 0    60   Output ~ 0
+RESET
+Wire Wire Line
+	1150 2400 2400 2400
+Wire Wire Line
+	1150 2500 2400 2500
+Wire Wire Line
+	2900 1500 2900 2000
+Wire Wire Line
+	2100 1600 3000 1600
+Connection ~ 2900 1600
+Wire Wire Line
+	3800 2700 3800 1500
+Wire Wire Line
+	3400 2700 3800 2700
+Wire Wire Line
+	2900 3200 2900 3000
+Wire Wire Line
+	1700 1600 1800 1600
+Wire Wire Line
+	2400 2400 2400 1900
+Wire Wire Line
+	2200 1900 2200 2000
+Wire Wire Line
+	2200 2000 2300 2000
+Wire Wire Line
+	2300 2000 2300 2500
+Connection ~ 2300 2500
+Connection ~ 2400 1600
+Connection ~ 2200 1600
+Wire Wire Line
+	9400 2600 9800 2600
+Wire Wire Line
+	9400 2300 10400 2300
+Wire Wire Line
+	9600 2300 9600 2700
+Wire Wire Line
+	9600 2700 9800 2700
+Wire Wire Line
+	9000 3000 9000 3200
+Wire Wire Line
+	9800 2800 9600 2800
+Wire Wire Line
+	9600 2800 9600 3100
+Wire Wire Line
+	9000 3100 10300 3100
+Connection ~ 9000 3100
+Wire Wire Line
+	9000 1700 9000 1900
+Wire Wire Line
+	9300 1800 9000 1800
+Connection ~ 9000 1800
+Wire Wire Line
+	9600 1800 9700 1800
+Wire Wire Line
+	9700 1800 9700 1900
+Wire Wire Line
+	8600 2400 8600 2500
+Wire Wire Line
+	5850 2800 5850 2700
+Wire Wire Line
+	5850 2700 5950 2700
+Wire Wire Line
+	8400 2300 8600 2300
+Wire Wire Line
+	8600 2400 8400 2400
+Wire Wire Line
+	8400 2600 8600 2600
+Wire Wire Line
+	10300 3100 10300 2800
+Connection ~ 9600 3100
+Wire Wire Line
+	10300 2600 10300 2450
+Wire Wire Line
+	10300 2450 9800 2450
+Wire Wire Line
+	9800 2450 9800 2600
+Wire Wire Line
+	10300 2700 10400 2700
+Wire Wire Line
+	10400 2700 10400 2300
+Connection ~ 9600 2300
+Wire Wire Line
+	5400 1900 5800 1900
+Wire Wire Line
+	5800 2200 5950 2200
+Wire Wire Line
+	5600 2300 5950 2300
+Wire Wire Line
+	5950 2400 5600 2400
+Wire Wire Line
+	4900 1800 4900 2500
+Wire Wire Line
+	4900 2500 5950 2500
+Wire Wire Line
+	2050 5100 1400 5100
+Wire Wire Line
+	1400 5100 1400 2400
+Connection ~ 1400 2400
+Wire Wire Line
+	2050 4900 1600 4900
+Wire Wire Line
+	1600 4900 1600 2500
+Connection ~ 1600 2500
+Wire Wire Line
+	2900 4600 2900 4250
+Wire Wire Line
+	2900 4400 3850 4400
+Wire Wire Line
+	3850 4400 3850 4450
+Connection ~ 2900 4400
+Wire Wire Line
+	3850 4750 3850 4800
+Wire Wire Line
+	2900 5900 2900 5800
+Wire Wire Line
+	2050 5400 2050 5850
+Wire Wire Line
+	2050 5850 2900 5850
+Connection ~ 2900 5850
+Connection ~ 2050 5600
+Connection ~ 2050 5500
+Wire Wire Line
+	3400 2500 3600 2500
+Wire Wire Line
+	3600 2500 3600 1500
+Wire Wire Line
+	3300 1600 3600 1600
+Connection ~ 3600 1600
 Wire Wire Line
 	3400 2400 3400 1800
@@
 	3000 1800 2900 1800
 Connection ~ 2900 1800
-Text HLabel 2100 2850 0    60   Output ~ 0
-RESET
-Wire Wire Line
-	2100 2850 2350 2850
-Wire Wire Line
-	2350 2850 2350 2700
-Connection ~ 2350 2700
+Wire Wire Line
+	1150 2700 2400 2700
 $EndSCHEMATC

Commit message: Added disconnect on DS323x reset line
Parts:
- added SB2: GS2, Connectors:GS2, symbol GS2
Connections:
- net RESET: now also SB2.1 (G1); no longer U6.4 (~RST)
- new net: SB2.2 (G2), U6.4 (~RST)
Changed lines of the file:
@@
 	3000 1800 2900 1800
 Connection ~ 2900 1800
+$Comp
+L GS2 SB2
+U 1 1 5A9B3265
+P 1900 2700
+F 0 "SB2" H 2000 2850 50  0000 C CNN
+F 1 "GS2" H 2000 2551 50  0000 C CNN
+F 2 "Connectors:GS2" V 1974 2700 50  0001 C CNN
+F 3 "" H 1900 2700 50  0001 C CNN
+	1    1900 2700
+	0    -1   -1   0
+$EndComp
 Wire Wire Line
-	1150 2700 2400 2700
+	1150 2700 1700 2700
+Wire Wire Line
+	2100 2700 2400 2700
 $EndSCHEMATC

Commit message: Added MSOP footprint for temp sensor
Parts:
- added U8: MCP9804_MSOP, Housings_SSOP:MSOP-8_3x3mm_Pitch0.65mm, symbol MCP9804_MSOP
- renumbered U8 to U9
Connections:
- net +3V3: now also U8.8 (VDD)
- net GND: now also U8.4 (GND), U8.5 (A2), U8.6 (A1), U8.7 (A0)
- net I2C1_SCL: now also U8.2 (SCL)
- net I2C1_SDA: now also U8.1 (SDA)
Other:
- moved on the sheet: C24
Changed lines of the file:
@@
 $EndComp
 $Comp
-L MAX485E U8
+L MAX485E U9
 U 1 1 5A0ADC38
 P 9000 2400
-F 0 "U8" H 8760 2850 50  0000 C CNN
+F 0 "U9" H 8760 2850 50  0000 C CNN
 F 1 "MAX485E" H 9030 2850 50  0000 L CNN
 F 2 "Housings_SOIC:SOIC-8_3.9x4.9mm_Pitch1.27mm" H 9000 1700 50  0001 C CNN
@@
 Text HLabel 5400 1900 0    60   Output ~ 0
 RESET
-Text HLabel 1150 2400 0    60   Input ~ 0
+Text HLabel 1400 2400 0    60   Input ~ 0
 I2C1_SCL
-Text HLabel 1150 2500 0    60   BiDi ~ 0
+Text HLabel 1400 2500 0    60   BiDi ~ 0
 I2C1_SDA
 Text HLabel 5600 2300 0    60   Input ~ 0
@@
 L C C24
 U 1 1 5A6AC90E
-P 3850 4600
-F 0 "C24" H 3875 4700 50  0000 L CNN
-F 1 "100 nF" H 3875 4500 50  0000 L CNN
-F 2 "Capacitors_SMD:C_0805" H 3888 4450 50  0001 C CNN
-F 3 "" H 3850 4600 50  0001 C CNN
-	1    3850 4600
+P 4150 4650
+F 0 "C24" H 4175 4750 50  0000 L CNN
+F 1 "100 nF" H 4175 4550 50  0000 L CNN
+F 2 "Capacitors_SMD:C_0805" H 4188 4500 50  0001 C CNN
+F 3 "" H 4150 4650 50  0001 C CNN
+	1    4150 4650
 	-1   0    0    1
 $EndComp
@@
 L GND #PWR046
 U 1 1 5A6ACBF8
-P 3850 4800
-F 0 "#PWR046" H 3850 4550 50  0001 C CNN
-F 1 "GND" H 3850 4650 50  0000 C CNN
-F 2 "" H 3850 4800 50  0001 C CNN
-F 3 "" H 3850 4800 50  0001 C CNN
-	1    3850 4800
+P 4150 4850
+F 0 "#PWR046" H 4150 4600 50  0001 C CNN
+F 1 "GND" H 4150 4700 50  0000 C CNN
+F 2 "" H 4150 4850 50  0001 C CNN
+F 3 "" H 4150 4850 50  0001 C CNN
+	1    4150 4850
 	1    0    0    -1
 $EndComp
@@
 	0    -1   -1   0
 $EndComp
-Text HLabel 1150 2700 0    60   Output ~ 0
+Text HLabel 1400 2700 0    60   Output ~ 0
 RESET
-Wire Wire Line
-	1150 2400 2400 2400
-Wire Wire Line
-	1150 2500 2400 2500
-Wire Wire Line
-	2900 1500 2900 2000
-Wire Wire Line
-	2100 1600 3000 1600
-Connection ~ 2900 1600
-Wire Wire Line
-	3800 2700 3800 1500
-Wire Wire Line
-	3400 2700 3800 2700
-Wire Wire Line
-	2900 3200 2900 3000
-Wire Wire Line
-	1700 1600 1800 1600
-Wire Wire Line
-	2400 2400 2400 1900
-Wire Wire Line
-	2200 1900 2200 2000
-Wire Wire Line
-	2200 2000 2300 2000
-Wire Wire Line
-	2300 2000 2300 2500
-Connection ~ 2300 2500
-Connection ~ 2400 1600
-Connection ~ 2200 1600
-Wire Wire Line
-	9400 2600 9800 2600
-Wire Wire Line
-	9400 2300 10400 2300
-Wire Wire Line
-	9600 2300 9600 2700
-Wire Wire Line
-	9600 2700 9800 2700
-Wire Wire Line
-	9000 3000 9000 3200
-Wire Wire Line
-	9800 2800 9600 2800
-Wire Wire Line
-	9600 2800 9600 3100
-Wire Wire Line
-	9000 3100 10300 3100
-Connection ~ 9000 3100
-Wire Wire Line
-	9000 1700 9000 1900
-Wire Wire Line
-	9300 1800 9000 1800
-Connection ~ 9000 1800
-Wire Wire Line
-	9600 1800 9700 1800
-Wire Wire Line
-	9700 1800 9700 1900
-Wire Wire Line
-	8600 2400 8600 2500
-Wire Wire Line
-	5850 2800 5850 2700
-Wire Wire Line
-	5850 2700 5950 2700
-Wire Wire Line
-	8400 2300 8600 2300
-Wire Wire Line
-	8600 2400 8400 2400
-Wire Wire Line
-	8400 2600 8600 2600
-Wire Wire Line
-	10300 3100 10300 2800
-Connection ~ 9600 3100
-Wire Wire Line
-	10300 2600 10300 2450
-Wire Wire Line
-	10300 2450 9800 2450
-Wire Wire Line
-	9800 2450 9800 2600
-Wire Wire Line
-	10300 2700 10400 2700
-Wire Wire Line
-	10400 2700 10400 2300
-Connection ~ 9600 2300
-Wire Wire Line
-	5400 1900 5800 1900
-Wire Wire Line
-	5800 2200 5950 2200
-Wire Wire Line
-	5600 2300 5950 2300
-Wire Wire Line
-	5950 2400 5600 2400
-Wire Wire Line
-	4900 1800 4900 2500
-Wire Wire Line
-	4900 2500 5950 2500
-Wire Wire Line
-	2050 5100 1400 5100
-Wire Wire Line
-	1400 5100 1400 2400
-Connection ~ 1400 2400
-Wire Wire Line
-	2050 4900 1600 4900
-Wire Wire Line
-	1600 4900 1600 2500
-Connection ~ 1600 2500
-Wire Wire Line
-	2900 4600 2900 4250
-Wire Wire Line
-	2900 4400 3850 4400
-Wire Wire Line
-	3850 4400 3850 4450
-Connection ~ 2900 4400
-Wire Wire Line
-	3850 4750 3850 4800
-Wire Wire Line
-	2900 5900 2900 5800
-Wire Wire Line
-	2050 5400 2050 5850
-Wire Wire Line
-	2050 5850 2900 5850
-Connection ~ 2900 5850
-Connection ~ 2050 5600
-Connection ~ 2050 5500
-Wire Wire Line
-	3400 2500 3600 2500
-Wire Wire Line
-	3600 2500 3600 1500
-Wire Wire Line
-	3300 1600 3600 1600
-Connection ~ 3600 1600
-Wire Wire Line
-	3400 2400 3400 1800
-Wire Wire Line
-	3400 1800 3300 1800
-Wire Wire Line
-	3000 1800 2900 1800
-Connection ~ 2900 1800
 $Comp
 L GS2 SB2
@@
 	0    -1   -1   0
 $EndComp
-Wire Wire Line
-	1150 2700 1700 2700
+$Comp
+L MCP9804_MSOP U8
+U 1 1 5AB87DF3
+P 6100 5100
+F 0 "U8" H 5850 5550 50  0000 C CNN
+F 1 "MCP9804_MSOP" H 6500 5550 50  0000 C CNN
+F 2 "Housings_SSOP:MSOP-8_3x3mm_Pitch0.65mm" H 5100 4600 50  0001 C CNN
+F 3 "" H 5850 5550 50  0001 C CNN
+	1    6100 5100
+	1    0    0    -1
+$EndComp
+Text HLabel 1400 5100 0    60   Input ~ 0
+I2C1_SCL
+Text HLabel 1400 4900 0    60   BiDi ~ 0
+I2C1_SDA
+Text HLabel 5200 4900 0    60   Input ~ 0
+I2C1_SCL
+Text HLabel 5200 4800 0    60   BiDi ~ 0
+I2C1_SDA
+Wire Wire Line
+	2900 1500 2900 2000
+Wire Wire Line
+	2100 1600 3000 1600
+Connection ~ 2900 1600
+Wire Wire Line
+	3800 2700 3800 1500
+Wire Wire Line
+	3400 2700 3800 2700
+Wire Wire Line
+	2900 3200 2900 3000
+Wire Wire Line
+	1700 1600 1800 1600
+Wire Wire Line
+	2400 1900 2400 2400
+Wire Wire Line
+	2200 1900 2200 2000
+Wire Wire Line
+	2200 2000 2300 2000
+Wire Wire Line
+	2300 2000 2300 2500
+Connection ~ 2400 1600
+Connection ~ 2200 1600
+Wire Wire Line
+	9400 2600 9800 2600
+Wire Wire Line
+	9400 2300 10400 2300
+Wire Wire Line
+	9600 2300 9600 2700
+Wire Wire Line
+	9600 2700 9800 2700
+Wire Wire Line
+	9000 3000 9000 3200
+Wire Wire Line
+	9800 2800 9600 2800
+Wire Wire Line
+	9600 2800 9600 3100
+Wire Wire Line
+	9000 3100 10300 3100
+Connection ~ 9000 3100
+Wire Wire Line
+	9000 1700 9000 1900
+Wire Wire Line
+	9300 1800 9000 1800
+Connection ~ 9000 1800
+Wire Wire Line
+	9600 1800 9700 1800
+Wire Wire Line
+	9700 1800 9700 1900
+Wire Wire Line
+	8600 2400 8600 2500
+Wire Wire Line
+	5850 2800 5850 2700
+Wire Wire Line
+	5850 2700 5950 2700
+Wire Wire Line
+	8400 2300 8600 2300
+Wire Wire Line
+	8600 2400 8400 2400
+Wire Wire Line
+	8400 2600 8600 2600
+Wire Wire Line
+	10300 3100 10300 2800
+Connection ~ 9600 3100
+Wire Wire Line
+	10300 2600 10300 2450
+Wire Wire Line
+	10300 2450 9800 2450
+Wire Wire Line
+	9800 2450 9800 2600
+Wire Wire Line
+	10300 2700 10400 2700
+Wire Wire Line
+	10400 2700 10400 2300
+Connection ~ 9600 2300
+Wire Wire Line
+	5400 1900 5800 1900
+Wire Wire Line
+	5800 2200 5950 2200
+Wire Wire Line
+	5600 2300 5950 2300
+Wire Wire Line
+	5950 2400 5600 2400
+Wire Wire Line
+	4900 1800 4900 2500
+Wire Wire Line
+	4900 2500 5950 2500
+Wire Wire Line
+	2900 4600 2900 4250
+Wire Wire Line
+	4150 4800 4150 4850
+Wire Wire Line
+	2900 5900 2900 5800
+Wire Wire Line
+	2050 5400 2050 5850
+Wire Wire Line
+	2050 5850 6100 5850
+Connection ~ 2900 5850
+Connection ~ 2050 5600
+Connection ~ 2050 5500
+Wire Wire Line
+	3400 2500 3600 2500
+Wire Wire Line
+	3600 2500 3600 1500
+Wire Wire Line
+	3300 1600 3600 1600
+Connection ~ 3600 1600
+Wire Wire Line
+	3400 2400 3400 1800
+Wire Wire Line
+	3400 1800 3300 1800
+Wire Wire Line
+	3000 1800 2900 1800
+Connection ~ 2900 1800
 Wire Wire Line
 	2100 2700 2400 2700
+Wire Wire Line
+	2400 2400 1400 2400
+Wire Wire Line
+	1400 2500 2400 2500
+Connection ~ 2300 2500
+Wire Wire Line
+	1700 2700 1400 2700
+Wire Wire Line
+	5200 4800 5700 4800
+Wire Wire Line
+	5700 4900 5200 4900
+Wire Wire Line
+	2050 4900 1400 4900
+Wire Wire Line
+	1400 5100 2050 5100
+Wire Wire Line
+	6100 4600 6100 4400
+Wire Wire Line
+	6100 4400 2900 4400
+Connection ~ 2900 4400
+Wire Wire Line
+	4150 4500 4150 4400
+Connection ~ 4150 4400
+Wire Wire Line
+	6100 5850 6100 5600
+Wire Wire Line
+	5700 5200 5700 5850
+Connection ~ 5700 5300
+Connection ~ 5700 5850
+Connection ~ 5700 5400
 $EndSCHEMATC

Commit message: Updated for KiCad v5, updated silks
Parts:
- C23, C24, C25, C26: symbol C -> Device:C
- J2: symbol Conn_01x06 -> kbxBinaryClock.v2.1-rescue:Conn_01x06
- J3: symbol Conn_02x03_Odd_Even -> kbxBinaryClock.v2.1-rescue:Conn_02x03_Odd_Even
- R38, R39, R40, R41: symbol R -> Device:R
- SB2: symbol GS2 -> win:GS2
- U6: symbol DS3231 -> kbxBinaryClock.v2.1-rescue:DS3231
- U7: symbol DS1621 -> kbxBinaryClock.v2.1-rescue:DS1621
- U8: symbol MCP9804_MSOP -> kbxBinaryClock.v2.1-rescue:MCP9804_MSOP
- U9: symbol MAX485E -> kbxBinaryClock.v2.1-rescue:MAX485E
Changed lines of the file:
@@
-EESchema Schematic File Version 2
-LIBS:power
-LIBS:device
-LIBS:transistors
-LIBS:conn
-LIBS:linear
-LIBS:regul
-LIBS:74xx
-LIBS:cmos4000
-LIBS:adc-dac
-LIBS:memory
-LIBS:xilinx
-LIBS:microcontrollers
-LIBS:dsp
-LIBS:microchip
-LIBS:analog_switches
-LIBS:motorola
-LIBS:texas
-LIBS:intel
-LIBS:audio
-LIBS:interface
-LIBS:digital-audio
-LIBS:philips
-LIBS:display
-LIBS:cypress
-LIBS:siliconi
-LIBS:opto
-LIBS:atmel
-LIBS:contrib
-LIBS:valves
-LIBS:stm32
-LIBS:win
-LIBS:mechanical
-LIBS:switches
-LIBS:maxim
-LIBS:sensors
+EESchema Schematic File Version 4
 LIBS:kbxBinaryClock.v2.1-cache
-EELAYER 25 0
+EELAYER 26 0
 EELAYER END
 $Descr A4 11693 8268
@@
 $EndDescr
 $Comp
-L DS3231 U6
+L kbxBinaryClock.v2.1-rescue:DS3231 U6
 U 1 1 5A0ADBD0
 P 2900 2500
@@
 $EndComp
 $Comp
-L MAX485E U9
+L kbxBinaryClock.v2.1-rescue:MAX485E U9
 U 1 1 5A0ADC38
 P 9000 2400
@@
 OSC32_IN
 $Comp
-L +3.3V #PWR036
+L power:+3.3V #PWR036
 U 1 1 5A0B2F0C
 P 2900 1500
@@
 $EndComp
 $Comp
-L R R40
+L Device:R R40
 U 1 1 5A0B2F28
 P 3150 1600
@@
 $EndComp
 $Comp
-L +BATT #PWR037
+L power:+BATT #PWR037
 U 1 1 5A0B2F97
 P 3800 1500
@@
 $EndComp
 $Comp
-L GND #PWR038
+L power:GND #PWR038
 U 1 1 5A0B2FCB
 P 2900 3200
@@
 $EndComp
 $Comp
-L C C23
+L Device:C C23
 U 1 1 5A0B2FFD
 P 1950 1600
@@
 $EndComp
 $Comp
-L GND #PWR039
+L power:GND #PWR039
 U 1 1 5A0B3065
 P 1700 1600
@@
 $EndComp
 $Comp
-L R R39
+L Device:R R39
 U 1 1 5A0B3562
 P 2400 1750
@@
 $EndComp
 $Comp
-L R R38
+L Device:R R38
 U 1 1 5A0B35AA
 P 2200 1750
@@
 $EndComp
 $Comp
-L GND #PWR040
+L power:GND #PWR040
 U 1 1 5A0B3A49
 P 9000 3200
@@
 $EndComp
 $Comp
-L +3.3V #PWR041
+L power:+3.3V #PWR041
 U 1 1 5A0B3ACB
 P 9000 1700
@@
 $EndComp
 $Comp
-L C C26
+L Device:C C26
 U 1 1 5A0B3B29
 P 9450 1800
@@
 $EndComp
 $Comp
-L GND #PWR042
+L power:GND #PWR042
 U 1 1 5A0B3BC0
 P 9700 1900
@@
 $EndComp
 $Comp
-L Conn_01x06 J2
+L kbxBinaryClock.v2.1-rescue:Conn_01x06 J2
 U 1 1 5A0B47CF
 P 6150 2500
@@
 $EndComp
 $Comp
-L GND #PWR043
+L power:GND #PWR043
 U 1 1 5A0B4904
 P 5850 2800
@@
 $EndComp
 $Comp
-L +3.3V #PWR044
+L power:+3.3V #PWR044
 U 1 1 5A0B49D6
 P 4900 1800
@@
 USART2_TX
 $Comp
-L Conn_02x03_Odd_Even J3
+L kbxBinaryClock.v2.1-rescue:Conn_02x03_Odd_Even J3
 U 1 1 5A0E0EE5
 P 10000 2700
@@
 $EndComp
 $Comp
-L C C25
+L Device:C C25
 U 1 1 5A6187BF
 P 5800 2050
@@
 $EndComp
 $Comp
-L DS1621 U7
+L kbxBinaryClock.v2.1-rescue:DS1621 U7
 U 1 1 5A6AC3DF
 P 2900 5200
@@
 $EndComp
 $Comp
-L +3.3V #PWR045
+L power:+3.3V #PWR045
 U 1 1 5A6AC87F
 P 2900 4250
@@
 $EndComp
 $Comp
-L C C24
+L Device:C C24
 U 1 1 5A6AC90E
 P 4150 4650
@@
 $EndComp
 $Comp
-L GND #PWR046
+L power:GND #PWR046
 U 1 1 5A6ACBF8
 P 4150 4850
@@
 $EndComp
 $Comp
-L GND #PWR047
+L power:GND #PWR047
 U 1 1 5A6ACE92
 P 2900 5900
@@
 $EndComp
 $Comp
-L R R41
+L Device:R R41
 U 1 1 5A800EAE
 P 3150 1800
@@
 RESET
 $Comp
-L GS2 SB2
+L win:GS2 SB2
 U 1 1 5A9B3265
 P 1900 2700
@@
 $EndComp
 $Comp
-L MCP9804_MSOP U8
+L kbxBinaryClock.v2.1-rescue:MCP9804_MSOP U8
 U 1 1 5AB87DF3
 P 6100 5100
