File: hardware/kbxBinaryClock.v3/kbxBinaryClock-Display.v3.sch (KiCad schematic (older format))
At the start: 54 parts, among them Q10 Q_NPN_BCE, Q11 Q_NPN_BCE, Q6 Q_NPN_BCE, Q7 Q_NPN_BCE, Q8 Q_NPN_BCE, Q9 Q_NPN_BCE, U2 TLC5947, U3 TLC5947, U4 TLC5947

Commit message: Added BoM, hw README, PCB tweaks
Parts:
- U2, U3, U4: Part Number (none) -> TLC5947DAP
Changed lines of the file:
@@
 F 1 "TLC5947" H 2350 4900 50  0000 C CNN
 F 2 "Housings_SSOP:HTSSOP-32_6.1x11mm_Pitch0.65mm_ThermalPad" H 2350 4750 50  0001 C CNN
-F 3 "DOCUMENTATION" H 2350 4650 50  0001 C CNN
+F 3 "http://www.ti.com/lit/ds/symlink/tlc5947.pdf" H 2350 4650 50  0001 C CNN
+F 4 "TLC5947DAP" H 2350 4950 60  0001 C CNN "Part Number"
 	1    2350 4950
 	0    -1   -1   0
@@
 F 1 "TLC5947" H 5850 4900 50  0000 C CNN
 F 2 "Housings_SSOP:HTSSOP-32_6.1x11mm_Pitch0.65mm_ThermalPad" H 5850 4750 50  0001 C CNN
-F 3 "DOCUMENTATION" H 5850 4650 50  0001 C CNN
+F 3 "http://www.ti.com/lit/ds/symlink/tlc5947.pdf" H 5850 4650 50  0001 C CNN
+F 4 "TLC5947DAP" H 5850 4950 60  0001 C CNN "Part Number"
 	1    5850 4950
 	0    -1   -1   0
@@
 F 1 "TLC5947" H 9350 4900 50  0000 C CNN
 F 2 "Housings_SSOP:HTSSOP-32_6.1x11mm_Pitch0.65mm_ThermalPad" H 9350 4750 50  0001 C CNN
-F 3 "DOCUMENTATION" H 9350 4650 50  0001 C CNN
+F 3 "http://www.ti.com/lit/ds/symlink/tlc5947.pdf" H 9350 4650 50  0001 C CNN
+F 4 "TLC5947DAP" H 9350 4950 60  0001 C CNN "Part Number"
 	1    9350 4950
 	0    -1   -1   0
@@
 F 1 "LED_RGB_COMMON_ANODE" H 2200 675 50  0000 C CNN
 F 2 "LEDs:LED_D5.0mm-4" H 2225 1100 60  0001 C CNN
-F 3 "" H 2225 1100 60  0000 C CNN
+F 3 "https://www.adafruit.com/product/302" H 2225 1100 60  0001 C CNN
 	1    2200 950
 	1    0    0    -1
@@
 F 1 "LED_RGB_COMMON_ANODE" H 2200 1375 50  0000 C CNN
 F 2 "LEDs:LED_D5.0mm-4" H 2225 1800 60  0001 C CNN
-F 3 "" H 2225 1800 60  0000 C CNN
+F 3 "https://www.adafruit.com/product/302" H 2225 1800 60  0001 C CNN
 	1    2200 1650
 	1    0    0    -1
@@
 F 1 "LED_RGB_COMMON_ANODE" H 2200 2075 50  0000 C CNN
 F 2 "LEDs:LED_D5.0mm-4" H 2225 2500 60  0001 C CNN
-F 3 "" H 2225 2500 60  0000 C CNN
+F 3 "https://www.adafruit.com/product/302" H 2225 2500 60  0001 C CNN
 	1    2200 2350
 	1    0    0    -1
@@
 F 1 "LED_RGB_COMMON_ANODE" H 2200 2775 50  0000 C CNN
 F 2 "LEDs:LED_D5.0mm-4" H 2225 3200 60  0001 C CNN
-F 3 "" H 2225 3200 60  0000 C CNN
+F 3 "https://www.adafruit.com/product/302" H 2225 3200 60  0001 C CNN
 	1    2200 3050
 	1    0    0    -1
@@
 F 1 "LED_RGB_COMMON_ANODE" H 3400 675 50  0000 C CNN
 F 2 "LEDs:LED_D5.0mm-4" H 3425 1100 60  0001 C CNN
-F 3 "" H 3425 1100 60  0000 C CNN
+F 3 "https://www.adafruit.com/product/302" H 3425 1100 60  0001 C CNN
 	1    3400 950
 	1    0    0    -1
@@
 F 1 "LED_RGB_COMMON_ANODE" H 3400 1375 50  0000 C CNN
 F 2 "LEDs:LED_D5.0mm-4" H 3425 1800 60  0001 C CNN
-F 3 "" H 3425 1800 60  0000 C CNN
+F 3 "https://www.adafruit.com/product/302" H 3425 1800 60  0001 C CNN
 	1    3400 1650
 	1    0    0    -1
@@
 F 1 "LED_RGB_COMMON_ANODE" H 3400 2075 50  0000 C CNN
 F 2 "LEDs:LED_D5.0mm-4" H 3425 2500 60  0001 C CNN
-F 3 "" H 3425 2500 60  0000 C CNN
+F 3 "https://www.adafruit.com/product/302" H 3425 2500 60  0001 C CNN
 	1    3400 2350
 	1    0    0    -1
@@
 F 1 "LED_RGB_COMMON_ANODE" H 3400 2775 50  0000 C CNN
 F 2 "LEDs:LED_D5.0mm-4" H 3425 3200 60  0001 C CNN
-F 3 "" H 3425 3200 60  0000 C CNN
+F 3 "https://www.adafruit.com/product/302" H 3425 3200 60  0001 C CNN
 	1    3400 3050
 	1    0    0    -1
@@
 F 1 "LED_RGB_COMMON_ANODE" H 4900 675 50  0000 C CNN
 F 2 "LEDs:LED_D5.0mm-4" H 4925 1100 60  0001 C CNN
-F 3 "" H 4925 1100 60  0000 C CNN
+F 3 "https://www.adafruit.com/product/302" H 4925 1100 60  0001 C CNN
 	1    4900 950
 	1    0    0    -1
@@
 F 1 "LED_RGB_COMMON_ANODE" H 4900 1375 50  0000 C CNN
 F 2 "LEDs:LED_D5.0mm-4" H 4925 1800 60  0001 C CNN
-F 3 "" H 4925 1800 60  0000 C CNN
+F 3 "https://www.adafruit.com/product/302" H 4925 1800 60  0001 C CNN
 	1    4900 1650
 	1    0    0    -1
@@
 F 1 "LED_RGB_COMMON_ANODE" H 4900 2075 50  0000 C CNN
 F 2 "LEDs:LED_D5.0mm-4" H 4925 2500 60  0001 C CNN
-F 3 "" H 4925 2500 60  0000 C CNN
+F 3 "https://www.adafruit.com/product/302" H 4925 2500 60  0001 C CNN
 	1    4900 2350
 	1    0    0    -1
@@
 F 1 "LED_RGB_COMMON_ANODE" H 4900 2775 50  0000 C CNN
 F 2 "LEDs:LED_D5.0mm-4" H 4925 3200 60  0001 C CNN
-F 3 "" H 4925 3200 60  0000 C CNN
+F 3 "https://www.adafruit.com/product/302" H 4925 3200 60  0001 C CNN
 	1    4900 3050
 	1    0    0    -1
@@
 F 1 "LED_RGB_COMMON_ANODE" H 6100 675 50  0000 C CNN
 F 2 "LEDs:LED_D5.0mm-4" H 6125 1100 60  0001 C CNN
-F 3 "" H 6125 1100 60  0000 C CNN
+F 3 "https://www.adafruit.com/product/302" H 6125 1100 60  0001 C CNN
 	1    6100 950
 	1    0    0    -1
@@
 F 1 "LED_RGB_COMMON_ANODE" H 6100 1375 50  0000 C CNN
 F 2 "LEDs:LED_D5.0mm-4" H 6125 1800 60  0001 C CNN
-F 3 "" H 6125 1800 60  0000 C CNN
+F 3 "https://www.adafruit.com/product/302" H 6125 1800 60  0001 C CNN
 	1    6100 1650
 	1    0    0    -1
@@
 F 1 "LED_RGB_COMMON_ANODE" H 6100 2075 50  0000 C CNN
 F 2 "LEDs:LED_D5.0mm-4" H 6125 2500 60  0001 C CNN
-F 3 "" H 6125 2500 60  0000 C CNN
+F 3 "https://www.adafruit.com/product/302" H 6125 2500 60  0001 C CNN
 	1    6100 2350
 	1    0    0    -1
@@
 F 1 "LED_RGB_COMMON_ANODE" H 6100 2775 50  0000 C CNN
 F 2 "LEDs:LED_D5.0mm-4" H 6125 3200 60  0001 C CNN
-F 3 "" H 6125 3200 60  0000 C CNN
+F 3 "https://www.adafruit.com/product/302" H 6125 3200 60  0001 C CNN
 	1    6100 3050
 	1    0    0    -1
@@
 F 1 "LED_RGB_COMMON_ANODE" H 7600 675 50  0000 C CNN
 F 2 "LEDs:LED_D5.0mm-4" H 7625 1100 60  0001 C CNN
-F 3 "" H 7625 1100 60  0000 C CNN
+F 3 "https://www.adafruit.com/product/302" H 7625 1100 60  0001 C CNN
 	1    7600 950
 	1    0    0    -1
@@
 F 1 "LED_RGB_COMMON_ANODE" H 7600 1375 50  0000 C CNN
 F 2 "LEDs:LED_D5.0mm-4" H 7625 1800 60  0001 C CNN
-F 3 "" H 7625 1800 60  0000 C CNN
+F 3 "https://www.adafruit.com/product/302" H 7625 1800 60  0001 C CNN
 	1    7600 1650
 	1    0    0    -1
@@
 F 1 "LED_RGB_COMMON_ANODE" H 7600 2075 50  0000 C CNN
 F 2 "LEDs:LED_D5.0mm-4" H 7625 2500 60  0001 C CNN
-F 3 "" H 7625 2500 60  0000 C CNN
+F 3 "https://www.adafruit.com/product/302" H 7625 2500 60  0001 C CNN
 	1    7600 2350
 	1    0    0    -1
@@
 F 1 "LED_RGB_COMMON_ANODE" H 7600 2775 50  0000 C CNN
 F 2 "LEDs:LED_D5.0mm-4" H 7625 3200 60  0001 C CNN
-F 3 "" H 7625 3200 60  0000 C CNN
+F 3 "https://www.adafruit.com/product/302" H 7625 3200 60  0001 C CNN
 	1    7600 3050
 	1    0    0    -1
@@
 F 1 "LED_RGB_COMMON_ANODE" H 8800 675 50  0000 C CNN
 F 2 "LEDs:LED_D5.0mm-4" H 8825 1100 60  0001 C CNN
-F 3 "" H 8825 1100 60  0000 C CNN
+F 3 "https://www.adafruit.com/product/302" H 8825 1100 60  0001 C CNN
 	1    8800 950
 	1    0    0    -1
@@
 F 1 "LED_RGB_COMMON_ANODE" H 8800 1375 50  0000 C CNN
 F 2 "LEDs:LED_D5.0mm-4" H 8825 1800 60  0001 C CNN
-F 3 "" H 8825 1800 60  0000 C CNN
+F 3 "https://www.adafruit.com/product/302" H 8825 1800 60  0001 C CNN
 	1    8800 1650
 	1    0    0    -1
@@
 F 1 "LED_RGB_COMMON_ANODE" H 8800 2075 50  0000 C CNN
 F 2 "LEDs:LED_D5.0mm-4" H 8825 2500 60  0001 C CNN
-F 3 "" H 8825 2500 60  0000 C CNN
+F 3 "https://www.adafruit.com/product/302" H 8825 2500 60  0001 C CNN
 	1    8800 2350
 	1    0    0    -1
@@
 F 1 "LED_RGB_COMMON_ANODE" H 8800 2775 50  0000 C CNN
 F 2 "LEDs:LED_D5.0mm-4" H 8825 3200 60  0001 C CNN
-F 3 "" H 8825 3200 60  0000 C CNN
+F 3 "https://www.adafruit.com/product/302" H 8825 3200 60  0001 C CNN
 	1    8800 3050
 	1    0    0    -1
@@
 F 1 "Q_NPN_BCE" H 6100 7050 50  0000 L CNN
 F 2 "TO_SOT_Packages_SMD:SOT-23" H 6700 7300 50  0001 C CNN
-F 3 "" H 6500 7200 50  0001 C CNN
+F 3 "https://www.diodes.com/assets/Datasheets/ds30036.pdf" H 6500 7200 50  0001 C CNN
 	1    6500 7200
 	-1   0    0    -1
@@
 F 1 "Q_NPN_BCE" H 5500 7050 50  0000 L CNN
 F 2 "TO_SOT_Packages_SMD:SOT-23" H 6100 7300 50  0001 C CNN
-F 3 "" H 5900 7200 50  0001 C CNN
+F 3 "https://www.diodes.com/assets/Datasheets/ds30036.pdf" H 5900 7200 50  0001 C CNN
 	1    5900 7200
 	1    0    0    -1
@@
 F 1 "Q_NPN_BCE" H 4300 7050 50  0000 L CNN
 F 2 "TO_SOT_Packages_SMD:SOT-23" H 4900 7300 50  0001 C CNN
-F 3 "" H 4700 7200 50  0001 C CNN
+F 3 "https://www.diodes.com/assets/Datasheets/ds30036.pdf" H 4700 7200 50  0001 C CNN
 	1    4700 7200
 	-1   0    0    -1
@@
 F 1 "Q_NPN_BCE" H 3700 7050 50  0000 L CNN
 F 2 "TO_SOT_Packages_SMD:SOT-23" H 4300 7300 50  0001 C CNN
-F 3 "" H 4100 7200 50  0001 C CNN
+F 3 "https://www.diodes.com/assets/Datasheets/ds30036.pdf" H 4100 7200 50  0001 C CNN
 	1    4100 7200
 	1    0    0    -1
@@
 F 1 "Q_NPN_BCE" H 2700 7050 50  0000 L CNN
 F 2 "TO_SOT_Packages_SMD:SOT-23" H 3300 7300 50  0001 C CNN
-F 3 "" H 3100 7200 50  0001 C CNN
+F 3 "https://www.diodes.com/assets/Datasheets/ds30036.pdf" H 3100 7200 50  0001 C CNN
 	1    3100 7200
 	-1   0    0    -1
@@
 F 1 "Q_NPN_BCE" H 2100 7050 50  0000 L CNN
 F 2 "TO_SOT_Packages_SMD:SOT-23" H 2700 7300 50  0001 C CNN
-F 3 "" H 2500 7200 50  0001 C CNN
+F 3 "https://www.diodes.com/assets/Datasheets/ds30036.pdf" H 2500 7200 50  0001 C CNN
 	1    2500 7200
 	1    0    0    -1

Commit message: Updated for KiCad v5, updated silks
Parts:
- C17, C18, C19: symbol C -> kbxBinaryClock.v3-rescue:C
- LED1, LED10, LED11, LED12, LED13, LED14, LED15, LED16, LED17, LED18, LED19, LED2, LED20, LED21, LED22, LED23, LED24, LED3, LED4, LED5, LED6, LED7, LED8, LED9: symbol LED_RGB_COMMON_ANODE -> kbxBinaryClock.v3-rescue:LED_RGB_COMMON_ANODE
- Q10, Q11, Q6, Q7, Q8, Q9: symbol Q_NPN_BCE -> kbxBinaryClock.v3-rescue:Q_NPN_BCE
- R20, R21, R22, R23, R24, R25, R26, R27, R28, R29, R30, R31, R32, R33, R34, R35, R36, R37: symbol R -> kbxBinaryClock.v3-rescue:R
- U2, U3, U4: symbol TLC5947 -> kbxBinaryClock.v3-rescue:TLC5947
