File: hardware/kbxBinaryClock.v3/kbxBinaryClock-Peripherals.v3.sch (KiCad schematic (older format))
At the start: 12 parts, among them J3 Conn_01x06, J4 Conn_02x03_Odd_Even, U6 DS3234, U7 DS1722, U8 LM74, U9 MAX485E

Commit message: Added BoM, hw README, PCB tweaks
Parts:
- U8: Part Number (none) -> LM74CIMX-3/NOPB
- U9: Part Number (none) -> ST1480ACDR
- renumbered J3 to J2, J4 to J3
Other:
- note added: "Install DS1722 *OR* LM74 -- DO NOT INSTALL BOTH"
Changed lines of the file:
@@
 F 1 "MAX485E" H 9030 2850 50  0000 L CNN
 F 2 "Housings_SOIC:SOIC-8_3.9x4.9mm_Pitch1.27mm" H 9000 1700 50  0001 C CNN
-F 3 "" H 9000 2450 50  0001 C CNN
+F 3 "http://www.st.com/content/ccc/resource/technical/document/datasheet/81/93/fa/ed/87/47/46/00/CD00003136.pdf/files/CD00003136.pdf/jcr:content/translations/en.CD00003136.pdf" H 9000 2450 50  0001 C CNN
+F 4 "ST1480ACDR" H 9000 2400 60  0001 C CNN "Part Number"
 	1    9000 2400
 	1    0    0    -1
@@
 $EndComp
 $Comp
-L Conn_01x06 J3
+L Conn_01x06 J2
 U 1 1 5A0B47CF
 P 6150 2500
-F 0 "J3" H 6150 2800 50  0000 C CNN
+F 0 "J2" H 6150 2800 50  0000 C CNN
 F 1 "Conn_01x06" H 6150 2100 50  0000 C CNN
 F 2 "Pin_Headers:Pin_Header_Straight_1x06_Pitch2.54mm" H 6150 2500 50  0001 C CNN
@@
 USART2_TX
 $Comp
-L Conn_02x03_Odd_Even J4
+L Conn_02x03_Odd_Even J3
 U 1 1 5A0E0EE5
 P 10000 2700
-F 0 "J4" H 10050 2900 50  0000 C CNN
+F 0 "J3" H 10050 2900 50  0000 C CNN
 F 1 "Conn_02x03_Odd_Even" H 10050 2500 50  0000 C CNN
 F 2 "Pin_Headers:Pin_Header_Straight_2x03_Pitch2.54mm" H 10000 2700 50  0001 C CNN
@@
 F 1 "DS3234" H 3050 3100 60  0000 C CNN
 F 2 "Housings_SOIC:SO-20_12.8x7.5mm_Pitch1.27mm" H 2850 2400 60  0001 C CNN
-F 3 "" H 2850 2400 60  0000 C CNN
+F 3 "https://datasheets.maximintegrated.com/en/ds/DS3234.pdf" H 2850 2400 60  0001 C CNN
 F 4 "Maxim" H 2650 1650 60  0001 C CNN "Manufacturer"
 	1    2850 2400
@@
 F 1 "LM74" H 5700 4550 60  0000 C CNN
 F 2 "Housings_SOIC:SOIC-8_3.9x4.9mm_Pitch1.27mm" H 5550 4850 60  0001 C CNN
-F 3 "" H 5550 4850 60  0001 C CNN
+F 3 "http://www.ti.com/lit/ds/symlink/lm74.pdf" H 5550 4850 60  0001 C CNN
+F 4 "LM74CIMX-3/NOPB" H 5550 4850 60  0001 C CNN "Part Number"
 	1    5550 4850
 	1    0    0    -1
@@
 F 1 "DS1722" H 3050 4550 60  0000 C CNN
 F 2 "Housings_SOIC:SOIC-8_3.9x4.9mm_Pitch1.27mm" H 2850 4950 60  0001 C CNN
-F 3 "" H 2850 4950 60  0001 C CNN
+F 3 "https://datasheets.maximintegrated.com/en/ds/DS1722.pdf" H 2850 4950 60  0001 C CNN
 	1    2850 4950
 	1    0    0    -1
@@
 Wire Wire Line
 	2250 1950 1900 1950
+Text Notes 2800 6050 0    60   ~ 0
+Install DS1722 *OR* LM74 -- DO NOT INSTALL BOTH
 $EndSCHEMATC

Commit message: Added disconnect on DS323x reset line
Parts:
- added SB2: GS2, Connectors:GS2, symbol GS2
Connections:
- net RESET: now also SB2.1 (G1); no longer U6.6 (~RST~)
- new net: SB2.2 (G2), U6.6 (~RST~)
Changed lines of the file:
@@
 	1350 2550 2350 2550
-Wire Wire Line
-	1350 2450 2350 2450
 Wire Wire Line
 	2350 2950 2350 2850
@@
 Text Notes 2800 6050 0    60   ~ 0
 Install DS1722 *OR* LM74 -- DO NOT INSTALL BOTH
+$Comp
+L GS2 SB2
+U 1 1 5A9B217E
+P 1600 2450
+F 0 "SB2" H 1700 2600 50  0000 C CNN
+F 1 "GS2" H 1700 2301 50  0000 C CNN
+F 2 "Connectors:GS2" V 1674 2450 50  0001 C CNN
+F 3 "" H 1600 2450 50  0001 C CNN
+	1    1600 2450
+	0    -1   -1   0
+$EndComp
+Wire Wire Line
+	1350 2450 1400 2450
+Wire Wire Line
+	1800 2450 2350 2450
 $EndSCHEMATC

Commit message: Updated for KiCad v5, updated silks
Parts:
- C23, C24, C25, C26: symbol C -> kbxBinaryClock.v3-rescue:C
- J2: symbol Conn_01x06 -> kbxBinaryClock.v3-rescue:Conn_01x06
- J3: symbol Conn_02x03_Odd_Even -> kbxBinaryClock.v3-rescue:Conn_02x03_Odd_Even
- R38, R39: symbol R -> kbxBinaryClock.v3-rescue:R
- SB2: symbol GS2 -> kbxBinaryClock.v3-rescue:GS2
- U6: symbol DS3234 -> kbxBinaryClock.v3-rescue:DS3234
- U7: symbol DS1722 -> kbxBinaryClock.v3-rescue:DS1722
- U8: symbol LM74 -> kbxBinaryClock.v3-rescue:LM74
- U9: symbol MAX485E -> kbxBinaryClock.v3-rescue:MAX485E
Changed lines of the file:
@@
-EESchema Schematic File Version 2
-LIBS:power
-LIBS:device
-LIBS:transistors
-LIBS:conn
-LIBS:linear
-LIBS:regul
-LIBS:74xx
-LIBS:cmos4000
-LIBS:adc-dac
-LIBS:memory
-LIBS:xilinx
-LIBS:microcontrollers
-LIBS:dsp
-LIBS:microchip
-LIBS:analog_switches
-LIBS:motorola
-LIBS:texas
-LIBS:intel
-LIBS:audio
-LIBS:interface
-LIBS:digital-audio
-LIBS:philips
-LIBS:display
-LIBS:cypress
-LIBS:siliconi
-LIBS:opto
-LIBS:atmel
-LIBS:contrib
-LIBS:valves
-LIBS:stm32
-LIBS:win
-LIBS:mechanical
-LIBS:switches
-LIBS:maxim
-LIBS:sensors
+EESchema Schematic File Version 4
 LIBS:kbxBinaryClock.v3-cache
-EELAYER 25 0
+EELAYER 26 0
 EELAYER END
 $Descr A4 11693 8268
@@
 $EndDescr
 $Comp
-L MAX485E U9
+L kbxBinaryClock.v3-rescue:MAX485E U9
 U 1 1 5A0ADC38
 P 9000 2400
@@
 OSC32_IN
 $Comp
-L +3.3V #PWR036
+L kbxBinaryClock.v3-rescue:+3.3V #PWR036
 U 1 1 5A0B2F0C
 P 3800 1500
@@
 $EndComp
 $Comp
-L +BATT #PWR037
+L kbxBinaryClock.v3-rescue:+BATT #PWR037
 U 1 1 5A0B2F97
 P 2250 1750
@@
 $EndComp
 $Comp
-L GND #PWR038
+L kbxBinaryClock.v3-rescue:GND #PWR038
 U 1 1 5A0B2FCB
 P 3350 3100
@@
 $EndComp
 $Comp
-L C C23
+L kbxBinaryClock.v3-rescue:C C23
 U 1 1 5A0B2FFD
 P 1900 2100
@@
 $EndComp
 $Comp
-L +3.3V #PWR039
+L kbxBinaryClock.v3-rescue:+3.3V #PWR039
 U 1 1 5A0B3116
 P 1900 1750
@@
 $EndComp
 $Comp
-L R R39
+L kbxBinaryClock.v3-rescue:R R39
 U 1 1 5A0B3562
 P 3600 1950
@@
 $EndComp
 $Comp
-L R R38
+L kbxBinaryClock.v3-rescue:R R38
 U 1 1 5A0B35AA
 P 3600 1750
@@
 $EndComp
 $Comp
-L GND #PWR040
+L kbxBinaryClock.v3-rescue:GND #PWR040
 U 1 1 5A0B3A49
 P 9000 3200
@@
 $EndComp
 $Comp
-L +3.3V #PWR041
+L kbxBinaryClock.v3-rescue:+3.3V #PWR041
 U 1 1 5A0B3ACB
 P 9000 1700
@@
 $EndComp
 $Comp
-L C C26
+L kbxBinaryClock.v3-rescue:C C26
 U 1 1 5A0B3B29
 P 9450 1800
@@
 $EndComp
 $Comp
-L GND #PWR042
+L kbxBinaryClock.v3-rescue:GND #PWR042
 U 1 1 5A0B3BC0
 P 9700 1900
@@
 $EndComp
 $Comp
-L Conn_01x06 J2
+L kbxBinaryClock.v3-rescue:Conn_01x06 J2
 U 1 1 5A0B47CF
 P 6150 2500
@@
 $EndComp
 $Comp
-L GND #PWR043
+L kbxBinaryClock.v3-rescue:GND #PWR043
 U 1 1 5A0B4904
 P 5850 2800
@@
 $EndComp
 $Comp
-L +3.3V #PWR044
+L kbxBinaryClock.v3-rescue:+3.3V #PWR044
 U 1 1 5A0B49D6
 P 4900 1800
@@
 USART2_TX
 $Comp
-L Conn_02x03_Odd_Even J3
+L kbxBinaryClock.v3-rescue:Conn_02x03_Odd_Even J3
 U 1 1 5A0E0EE5
 P 10000 2700
@@
 $EndComp
 $Comp
-L C C25
+L kbxBinaryClock.v3-rescue:C C25
 U 1 1 5A6187BF
 P 5800 2050
@@
 $EndComp
 $Comp
-L +3.3V #PWR045
+L kbxBinaryClock.v3-rescue:+3.3V #PWR045
 U 1 1 5A6AC87F
 P 2950 4100
@@
 $EndComp
 $Comp
-L C C24
+L kbxBinaryClock.v3-rescue:C C24
 U 1 1 5A6AC90E
 P 3600 5350
@@
 $EndComp
 $Comp
-L GND #PWR046
+L kbxBinaryClock.v3-rescue:GND #PWR046
 U 1 1 5A6ACBF8
 P 3600 5600
@@
 $EndComp
 $Comp
-L DS3234 U6
+L kbxBinaryClock.v3-rescue:DS3234 U6
 U 1 1 5A7DBF61
 P 2850 2400
@@
 SPI1_MISO
 $Comp
-L GND #PWR047
+L kbxBinaryClock.v3-rescue:GND #PWR047
 U 1 1 5A0B3065
 P 1900 2250
@@
 SPI1_NSS_RTC
 $Comp
-L LM74 U8
+L kbxBinaryClock.v3-rescue:LM74 U8
 U 1 1 5A7E2809
 P 5550 4850
@@
 Connection ~ 3600 4200
 $Comp
-L DS1722 U7
+L kbxBinaryClock.v3-rescue:DS1722 U7
 U 1 1 5A7E240D
 P 2850 4950
@@
 Install DS1722 *OR* LM74 -- DO NOT INSTALL BOTH
 $Comp
-L GS2 SB2
+L kbxBinaryClock.v3-rescue:GS2 SB2
 U 1 1 5A9B217E
 P 1600 2450
